File: design/eagle/frontend_v2.sch (EAGLE design)
At the start: 39 parts, among them U1 RF3865, U2 ALM32220

Commit message: design: Major revision of the PCB to fit into enclosure
Signed-off-by: Sylvain Munaut <tnt@246tNt.com>
Parts:
- removed L4, L5: 10n, we_passive:L-EU_0603
- removed R2, R3, R4: 0R, we_passive:R-EU_1210
- removed SV1: (no value), con-lstb-tnt:MA04-2SMD
- added C22, C24, C25, C26: 10u, rcl:CPOL-EUSMCA
- added C23: 22u, rcl:CPOL-EUSMCA
- added D1, D2, D3, D4, D5: PESD5V0F1BL, we_passive:D_ESD_SOD882
- added FB1, FB2: (no value), we_passive:FBEAD_1206
- added FB3, FB4: (no value), we_passive:FBEAD_0603
- added J1: DC_IN, con-molex:22-27-2021-02
- added J2: 5V_OUT, con-molex:22-27-2021-02
- added RX_OUT_UFL, TX_IN_UFL: (no value), we_conn:HRS_UFL
- added SHLD1: (no value), we_mech:SHIELD25X25
- added U3: MIC29301-5.0BT, we_chips:MIC29XXX-FIX_WT_TO220BV
- ANT, RX_OUT, TX_IN: device we_conn:SMA-F-S-EDGE -> we_conn:SMA-F-S-TH
- C11: value 10n -> 10p
- C14: value 100n -> 10n
- C15: value 2.2u -> 100n; device we_passive:C-EU_0805 -> we_passive:C-EU_0603
- C17: value 10n -> DNP
- C18: value 100n -> 10p
- C19: value 47u -> 10n; device rcl:CPOL-EUSMCA -> we_passive:C-EU_0603
- C2: value 15p -> 10n
- C20: value 47u -> 100n; device rcl:CPOL-EUSMCA -> we_passive:C-EU_0603
- C21: value 47u -> 2.2u; device rcl:CPOL-EUSMCA -> we_passive:C-EU_0805
- C4: value 10n -> 15p
- C5: value 100pF -> 100p
- C9: value 10p -> DNP
- L1: value DNP -> 27n
- L2: value DNP -> 10n
- L3: value 27n -> 10n
Connections:
- removed net N$13: R3.1, SV1.5
- removed net N$7: R2.1, SV1.7, SV1.8
- new net 5V: C23.+, FB2.1, FB3.1, FB4.1, J2-1.S, U3.VOUT
- new net DC_IN: FB1.1, J1-1.S
- new net DC_IN_FLT: C22.+, FB1.2, U3.VIN
- new net N$8: C10.2, D2.2, RX_OUT_UFL.1
- new net N$9: C10.1, C11.1, FLT3G.OUT
- net 5V_LNA: now also C26.+, FB4.2, L1.1, L2.1; no longer C21.+, L3.1, L4.1, R4.2
- net 5V_PA: now also C19.1, C20.1, C21.1, C24.+, FB2.2; no longer C11.1, C12.1, C13.1, C19.+, R2.2
- net 5V_PACTRL: now also C12.1, C13.1, C25.+, FB3.2; no longer C17.1, C18.1, C20.+, R3.2
- net GND: now also C19.2, C20.2, C21.2, C22.-, C23.-, C24.-, C25.-, C26.-, C9.2, D1.1, D2.1, D3.1, D4.1, D5.1, J1-2.S, J2-2.S, RX_OUT_UFL.GND@1, RX_OUT_UFL.GND@2, TX_IN_UFL.GND@1, TX_IN_UFL.GND@2, U3.GND; no longer C10.2, C11.2, C17.2, C18.2, C19.-, C20.-, C21.-, L1.2, L2.2, SV1.1, SV1.2, SV1.3, SV1.4
- net N$1: now also L1.2; no longer L3.2
- net N$10: now also L2.2; no longer L4.2
- net N$14: now also C17.1, D5.2, TX_IN_UFL.1; no longer R4.1, SV1.6
- net N$2: now also C18.1, D4.2; no longer C9.1
- net N$3: now also C17.2, C18.2; no longer C9.2
- net N$4: now also L3.2; no longer L5.2
- net N$6: now also C9.1; no longer C7.1
- net RF_ANT: now also D1.2; no longer L1.1
- net RF_UPLINK: now also L3.1; no longer L5.1
- net RF_UPLINK_IS_OUT: now also C7.1; no longer C10.1
- net RF_UPLINK_OUT: now also C11.2, D3.2; no longer FLT3G.OUT, L2.1
