File: design/eagle/pa_only_1800.brd (EAGLE design)
At the start: 76.2 x 88.9 mm, 53 parts, among them J1 DC_IN, J2 5V_OUT, U1 RF3865, U2 ALM32220, U3 MIC29301-5.0BT

Commit message: add a PA-only version without LNA for DCS 1800
Parts:
- removed C1, C2, L2, L3: 10n, we_passive:0603
- removed C26: 10u, rcl:SMC_A
- removed C3, C4: 15p, we_passive:0603
- removed C5: 100p, we_passive:0603
- removed C6: 10p, we_passive:0603
- removed C7, C8, C9, R1: DNP, we_passive:0603
- removed FB4: (no value), we_passive:0603
- removed FLT2, FLT3: EPCOS_B3832, we_passive:DCC6C
- removed L1: 27n, we_passive:0603
- removed SHLD1: (no value), we_mech:WE-SHC-SMD_25X25
- removed U1: RF3865, we_chips:QFN20_5X5_PAD
- moved J1 7.62 mm to (15.2, 84.5)
- moved J2 7.62 mm to (15.2, 76.8)
- moved U3 5.08 mm to (7.30, 80.6), turned to 270 degrees
- moved C22 5.08 mm to (8.89, 83.2), turned to 270 degrees
- moved C23 5.08 mm to (8.89, 78.1), turned to 90 degrees
- moved FB1 5.08 mm to (11.4, 83.2), turned to 90 degrees
Connections:
- removed net 5V_LNA: C1.1, C2.1, C26.+, C3.1, C4.1, FB4.2, L1.1, L2.1
- removed net N$1: L1.2, U1.19
- removed net N$10: L2.2, U1.17
- removed net N$4: C5.1, L3.2
- removed net N$5: C5.2, C6.1, U1.5
- removed net N$6: C9.1, R1.2, U1.11
- removed net N$9: C10.1, C11.1, FLT3.5
- removed net RF_UPLINK_IS_IN: C8.1, FLT2.5, U1.9
- removed net RF_UPLINK_IS_OUT: C7.1, FLT2.2, U1.7
- removed net RF_UPLINK_LNA_OUT: FLT3.2, U1.13
- net 5V: no longer FB4.1
- net GND: no longer C1.2, C2.2, C26.-, C3.2, C4.2, C6.2, C7.2, C8.2, C9.2, FLT2.1, FLT2.3, FLT2.4, FLT2.6, FLT3.1, FLT3.3, FLT3.4, FLT3.6, R1.1, U1.PAD
- net RF_UPLINK: now also C10.1, C11.1; no longer L3.1, U1.3
Routing:
- net 5V_LNA: track 100.4 -> 0.00 mm
- net RF_UPLINK: track 9.98 -> 33.2 mm
- net GND: track 39.0 -> 22.9 mm, vias 596 -> 501
- net RF_UPLINK_IS_OUT: track 11.5 -> 0.00 mm
- net RF_UPLINK_IS_IN: track 11.5 -> 0.00 mm
- net N$9: track 8.48 -> 0.00 mm
- net RF_UPLINK_LNA_OUT: track 6.70 -> 0.00 mm
- net 5V: track 38.5 -> 32.4 mm
- net N$6: track 3.15 -> 0.00 mm
- net N$5: track 3.13 -> 0.00 mm
- net N$4: track 1.97 -> 0.00 mm
- net N$10: track 1.81 -> 0.00 mm
- net N$1: track 1.81 -> 0.00 mm
- net DC_IN_FLT: track 11.9 -> 12.6 mm
Other:
- board text added: "D55413A"
- board text added: "osmo-bts-amp pa_only_1800"
- board text added: "v3 20121022"
- board text removed: "D51395A"
- board text removed: "osmo-bts-amp"
- board text removed: "v2.1 20120518"
