File: design/eagle/pa_only_900.brd (EAGLE design)
At the start: 76.2 x 88.9 mm, 34 parts, among them J1 DC_IN, J2 5V_OUT, U2 ALM32220, U3 MIC29301-5.0BT

Commit message: schematics / gerber of 900 MHz PA-only version
Parts:
- removed FLT1: RADITEK_RDUP-1710-1785M-1805-1880M-4415-3W-S-CA-J2, we_passive:RADITEK_RDUP_4415
- added U$3: RDUP-880-915M-925-960M-4217-3W-S-J, laforge:RADITEK_4217
Connections:
- net GND: now also U$3.G1, U$3.G2, U$3.G3, U$3.G4, U$3.G5, U$3.G6, U$3.G7; no longer FLT1.GND@1, FLT1.GND@10, FLT1.GND@11, FLT1.GND@12, FLT1.GND@13, FLT1.GND@14, FLT1.GND@15, FLT1.GND@2, FLT1.GND@3, FLT1.GND@4, FLT1.GND@5, FLT1.GND@6, FLT1.GND@7, FLT1.GND@8, FLT1.GND@9
- net RF_ANT: now also U$3.C; no longer FLT1.ANT
- net RF_DOWNLINK: now also U$3.H; no longer FLT1.HI
- net RF_UPLINK: now also U$3.L; no longer FLT1.LO
Routing:
- net RF_DOWNLINK: track 13.3 -> 15.1 mm
- net RF_UPLINK: track 33.2 -> 34.6 mm
- net RF_ANT: track 41.2 -> 42.5 mm
- net GND: vias 501 -> 508
Other:
- board text added: "D55413B"
- board text added: "osmo-bts-amp pa_only_900"
- board text removed: "D55413A"
- board text removed: "osmo-bts-amp pa_only_1800"
