File: design/eagle/pa_only_900.sch (EAGLE design)
At the start: 34 parts, among them J1 DC_IN, J2 5V_OUT, U2 ALM32220, U3 MIC29301-5.0BT

Commit message: schematics / gerber of 900 MHz PA-only version
Parts:
- removed FLT1: RADITEK_RDUP-1710-1785M-1805-1880M-4415-3W-S-CA-J2, we_passive:RADITEK_RDUP-1710-1785M-1805-1880M-4415-3W-S-CA-J2
- added U$3: RDUP-880-915M-925-960M-4217-3W-S-J, laforge:RDUP-880-915M-925-960M-4217-3W-S-J
Connections:
- net GND: now also U$3G$2.P$1, U$3G$2.P$2, U$3G$2.P$3, U$3G$2.P$4, U$3G$2.P$5, U$3G$2.P$6, U$3G$2.P$7; no longer FLT1CASE.GND@1, FLT1CASE.GND@10, FLT1CASE.GND@11, FLT1CASE.GND@12, FLT1CASE.GND@13, FLT1CASE.GND@14, FLT1CASE.GND@15, FLT1CASE.GND@2, FLT1CASE.GND@3, FLT1CASE.GND@4, FLT1CASE.GND@5, FLT1CASE.GND@6, FLT1CASE.GND@7, FLT1CASE.GND@8, FLT1CASE.GND@9
- net RF_ANT: now also U$3G$1.COM; no longer FLT1G.ANT
- net RF_DOWNLINK: now also U$3G$1.HI; no longer FLT1G.HI
- net RF_UPLINK: now also U$3G$1.LO; no longer FLT1G.LO
Changed lines of the file:
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@@
 </classes>
 <parts>
-<part name="FLT1" library="we_passive" deviceset="RADITEK_RDUP-1710-1785M-1805-1880M-4415-3W-S-CA-J2" device=""/>
 <part name="ANT" library="we_conn" deviceset="SMA-F" device="-S-TH"/>
 <part name="FRAME1" library="frames" deviceset="DINA4_L" device=""/>
@@
 <part name="U$44" library="we_supply" deviceset="GND" device=""/>
 <part name="U$45" library="we_supply" deviceset="GND" device=""/>
+<part name="U$3" library="laforge" deviceset="RDUP-880-915M-925-960M-4217-3W-S-J" device=""/>
 </parts>
 <sheets>
@@
 </plain>
 <instances>
-<instance part="FLT1" gate="G" x="127" y="116.84" smashed="yes">
-<attribute name="NAME" x="119.38" y="101.6" size="1.778" layer="95" font="vector" rot="MR180"/>
-<attribute name="VALUE" x="119.38" y="132.08" size="1.778" layer="96" font="vector"/>
-</instance>
-<instance part="FLT1" gate="CASE" x="55.88" y="58.42"/>
 <instance part="ANT" gate="G" x="73.66" y="116.84"/>
 <instance part="FRAME1" gate="G$1" x="0" y="0"/>
@@
 <instance part="D1" gate="SYM" x="88.9" y="101.6" rot="R90"/>
 <instance part="U$36" gate="G$1" x="88.9" y="91.44"/>
+<instance part="U$3" gate="G$1" x="129.54" y="116.84"/>
+<instance part="U$3" gate="G$2" x="53.34" y="60.96"/>
 </instances>
 <busses>
@@
 <net name="GND" class="0">
 <segment>
-<wire x1="38.1" y1="50.8" x2="38.1" y2="48.26" width="0.1524" layer="91"/>
-<wire x1="38.1" y1="48.26" x2="40.64" y2="48.26" width="0.1524" layer="91"/>
-<wire x1="40.64" y1="48.26" x2="43.18" y2="48.26" width="0.1524" layer="91"/>
-<wire x1="43.18" y1="48.26" x2="45.72" y2="48.26" width="0.1524" layer="91"/>
 <wire x1="45.72" y1="48.26" x2="48.26" y2="48.26" width="0.1524" layer="91"/>
 <wire x1="48.26" y1="48.26" x2="50.8" y2="48.26" width="0.1524" layer="91"/>
@@
 <wire x1="55.88" y1="48.26" x2="58.42" y2="48.26" width="0.1524" layer="91"/>
 <wire x1="58.42" y1="48.26" x2="60.96" y2="48.26" width="0.1524" layer="91"/>
-<wire x1="60.96" y1="48.26" x2="63.5" y2="48.26" width="0.1524" layer="91"/>
-<wire x1="63.5" y1="48.26" x2="66.04" y2="48.26" width="0.1524" layer="91"/>
-<wire x1="66.04" y1="48.26" x2="68.58" y2="48.26" width="0.1524" layer="91"/>
-<wire x1="68.58" y1="48.26" x2="71.12" y2="48.26" width="0.1524" layer="91"/>
-<wire x1="71.12" y1="48.26" x2="73.66" y2="48.26" width="0.1524" layer="91"/>
-<wire x1="73.66" y1="48.26" x2="73.66" y2="50.8" width="0.1524" layer="91"/>
 <wire x1="53.34" y1="50.8" x2="53.34" y2="48.26" width="0.1524" layer="91"/>
 <wire x1="53.34" y1="48.26" x2="53.34" y2="45.72" width="0.1524" layer="91"/>
-<wire x1="40.64" y1="50.8" x2="40.64" y2="48.26" width="0.1524" layer="91"/>
-<wire x1="43.18" y1="50.8" x2="43.18" y2="48.26" width="0.1524" layer="91"/>
 <wire x1="45.72" y1="50.8" x2="45.72" y2="48.26" width="0.1524" layer="91"/>
 <wire x1="48.26" y1="50.8" x2="48.26" y2="48.26" width="0.1524" layer="91"/>
@@
 <wire x1="58.42" y1="50.8" x2="58.42" y2="48.26" width="0.1524" layer="91"/>
 <wire x1="60.96" y1="50.8" x2="60.96" y2="48.26" width="0.1524" layer="91"/>
-<wire x1="63.5" y1="50.8" x2="63.5" y2="48.26" width="0.1524" layer="91"/>
-<wire x1="66.04" y1="50.8" x2="66.04" y2="48.26" width="0.1524" layer="91"/>
-<wire x1="68.58" y1="50.8" x2="68.58" y2="48.26" width="0.1524" layer="91"/>
-<wire x1="71.12" y1="50.8" x2="71.12" y2="48.26" width="0.1524" layer="91"/>
 <junction x="53.34" y="48.26"/>
-<junction x="40.64" y="48.26"/>
-<junction x="43.18" y="48.26"/>
-<junction x="45.72" y="48.26"/>
 <junction x="48.26" y="48.26"/>
 <junction x="50.8" y="48.26"/>
 <junction x="55.88" y="48.26"/>
 <junction x="58.42" y="48.26"/>
-<junction x="60.96" y="48.26"/>
-<junction x="63.5" y="48.26"/>
-<junction x="66.04" y="48.26"/>
-<junction x="68.58" y="48.26"/>
-<junction x="71.12" y="48.26"/>
-<pinref part="FLT1" gate="CASE" pin="GND@1"/>
-<pinref part="FLT1" gate="CASE" pin="GND@15"/>
-<pinref part="FLT1" gate="CASE" pin="GND@7"/>
 <pinref part="U$1" gate="G$1" pin="GND"/>
-<pinref part="FLT1" gate="CASE" pin="GND@2"/>
-<pinref part="FLT1" gate="CASE" pin="GND@3"/>
-<pinref part="FLT1" gate="CASE" pin="GND@4"/>
-<pinref part="FLT1" gate="CASE" pin="GND@5"/>
-<pinref part="FLT1" gate="CASE" pin="GND@6"/>
-<pinref part="FLT1" gate="CASE" pin="GND@8"/>
-<pinref part="FLT1" gate="CASE" pin="GND@9"/>
-<pinref part="FLT1" gate="CASE" pin="GND@10"/>
-<pinref part="FLT1" gate="CASE" pin="GND@11"/>
-<pinref part="FLT1" gate="CASE" pin="GND@12"/>
-<pinref part="FLT1" gate="CASE" pin="GND@13"/>
-<pinref part="FLT1" gate="CASE" pin="GND@14"/>
+<pinref part="U$3" gate="G$2" pin="P$1"/>
+<pinref part="U$3" gate="G$2" pin="P$2"/>
+<pinref part="U$3" gate="G$2" pin="P$3"/>
+<pinref part="U$3" gate="G$2" pin="P$4"/>
+<pinref part="U$3" gate="G$2" pin="P$5"/>
+<pinref part="U$3" gate="G$2" pin="P$6"/>
+<pinref part="U$3" gate="G$2" pin="P$7"/>
 </segment>
 <segment>
@@
 <net name="RF_ANT" class="0">
 <segment>
-<pinref part="FLT1" gate="G" pin="ANT"/>
 <pinref part="ANT" gate="G" pin="1"/>
 <wire x1="76.2" y1="116.84" x2="88.9" y2="116.84" width="0.1524" layer="91"/>
@@
 <wire x1="88.9" y1="106.68" x2="88.9" y2="116.84" width="0.1524" layer="91"/>
 <junction x="88.9" y="116.84"/>
-<wire x1="114.3" y1="116.84" x2="88.9" y2="116.84" width="0.1524" layer="91"/>
+<wire x1="116.84" y1="116.84" x2="88.9" y2="116.84" width="0.1524" layer="91"/>
+<pinref part="U$3" gate="G$1" pin="COM"/>
 </segment>
 </net>
 <net name="RF_DOWNLINK" class="0">
 <segment>
-<wire x1="139.7" y1="127" x2="165.1" y2="127" width="0.1524" layer="91"/>
+<wire x1="129.54" y1="129.54" x2="165.1" y2="129.54" width="0.1524" layer="91"/>
 <label x="144.78" y="129.54" size="1.778" layer="95" rot="MR180"/>
-<pinref part="FLT1" gate="G" pin="HI"/>
+<pinref part="U$3" gate="G$1" pin="HI"/>
 </segment>
 </net>
 <net name="RF_UPLINK" class="0">
 <segment>
-<wire x1="139.7" y1="106.68" x2="165.1" y2="106.68" width="0.1524" layer="91"/>
+<wire x1="129.54" y1="104.14" x2="165.1" y2="104.14" width="0.1524" layer="91"/>
 <label x="144.78" y="109.22" size="1.778" layer="95" rot="MR180"/>
-<pinref part="FLT1" gate="G" pin="LO"/>
+<pinref part="U$3" gate="G$1" pin="LO"/>
 </segment>
 </net>
